File: schematic/wearlink.sch (KiCad schematic (older format))
At the start: 8 parts, among them J1 JTAG, Q1 MMBT3904, U1 WT51822-0S4AT

Commit message: Added footprints, first route
Seems a little to spacious..
Parts:
- BT1: value Battery_Cell -> Battery 2032
- J1: footprint Connectors_Molex:Molex_KK-6410-04_04x2.54mm_Straight -> wearlink:TC2030-IDC-NL; symbol Conn_01x04 -> Conn_01x06
- R1, R2, R3: footprint Resistors_SMD:R_0805_HandSoldering -> Resistors_SMD:R_0603
- S1: footprint Connectors:Banana_Jack_3Pin -> Connectors_Molex:Molex_KK-6410-02_02x2.54mm_Straight
Connections:
- net labels added: GND
- wire segments 25 -> 30
Changed lines of the file:
@@
 LIBS:WT51822-0S4AT
 LIBS:fibretronickeypad
+LIBS:wearlink-cache
 EELAYER 25 0
 EELAYER END
@@
 U 1 1 5AED9A99
 P 2650 2950
-F 0 "BT1" H 2750 3050 50  0000 L CNN
-F 1 "Battery_Cell" H 2750 2950 50  0000 L CNN
+F 0 "BT1" H 2400 3050 50  0000 L CNN
+F 1 "Battery 2032" H 2150 2900 50  0000 L CNN
 F 2 "Battery_Holders:Keystone_3034_1x20mm-CoinCell" V 2650 3010 50  0001 C CNN
 F 3 "" V 2650 3010 50  0001 C CNN
@@
 L +3.3V #PWR01
 U 1 1 5AEDB4DB
-P 6350 1850
-F 0 "#PWR01" H 6350 1700 50  0001 C CNN
-F 1 "+3.3V" H 6350 1990 50  0000 C CNN
-F 2 "" H 6350 1850 50  0001 C CNN
-F 3 "" H 6350 1850 50  0001 C CNN
-	1    6350 1850
+P 4650 1850
+F 0 "#PWR01" H 4650 1700 50  0001 C CNN
+F 1 "+3.3V" H 4650 1990 50  0000 C CNN
+F 2 "" H 4650 1850 50  0001 C CNN
+F 3 "" H 4650 1850 50  0001 C CNN
+	1    4650 1850
 	1    0    0    -1
 $EndComp
@@
 F 0 "S1" H 9340 2730 60  0000 C CNN
 F 1 "FibretronicKeypad" H 8340 2730 60  0000 C CNN
-F 2 "Connectors:Banana_Jack_3Pin" H 8650 2350 60  0001 C CNN
+F 2 "Connectors_Molex:Molex_KK-6410-02_02x2.54mm_Straight" H 8650 2350 60  0001 C CNN
 F 3 "" H 8650 2350 60  0001 C CNN
 	1    8650 2350
@@
 F 0 "R1" V 6330 3550 50  0000 C CNN
 F 1 "20k" V 6250 3550 50  0000 C CNN
-F 2 "Resistors_SMD:R_0805_HandSoldering" V 6180 3550 50  0001 C CNN
+F 2 "Resistors_SMD:R_0603" V 6180 3550 50  0001 C CNN
 F 3 "" H 6250 3550 50  0001 C CNN
 	1    6250 3550
@@
 F 0 "R3" V 7130 2150 50  0000 C CNN
 F 1 "1M" V 7050 2150 50  0000 C CNN
-F 2 "Resistors_SMD:R_0805_HandSoldering" V 6980 2150 50  0001 C CNN
+F 2 "Resistors_SMD:R_0603" V 6980 2150 50  0001 C CNN
 F 3 "" H 7050 2150 50  0001 C CNN
 	1    7050 2150
@@
 F 0 "R2" V 6580 3200 50  0000 C CNN
 F 1 "1M" V 6500 3200 50  0000 C CNN
-F 2 "Resistors_SMD:R_0805_HandSoldering" V 6430 3200 50  0001 C CNN
+F 2 "Resistors_SMD:R_0603" V 6430 3200 50  0001 C CNN
 F 3 "" H 6500 3200 50  0001 C CNN
 	1    6500 3200
@@
 POWER
 $Comp
-L Conn_01x04 J1
+L Conn_01x06 J1
 U 1 1 5AEDCC20
-P 3400 3250
-F 0 "J1" H 3400 3450 50  0000 C CNN
-F 1 "JTAG" H 3400 2900 50  0000 C CNN
-F 2 "Connectors_Molex:Molex_KK-6410-04_04x2.54mm_Straight" H 3400 3250 50  0001 C CNN
-F 3 "" H 3400 3250 50  0001 C CNN
-	1    3400 3250
-	-1   0    0    1
-$EndComp
-Wire Wire Line
-	3600 3050 3600 1850
-Connection ~ 3600 1850
-Wire Wire Line
-	3600 3350 3600 4050
-Connection ~ 3600 4050
-Wire Wire Line
-	3600 3250 3850 3250
-Wire Wire Line
-	3600 3150 3850 3150
+P 3200 3050
+F 0 "J1" H 3200 3350 50  0000 C CNN
+F 1 "JTAG" H 3200 2650 50  0000 C CNN
+F 2 "wearlink:TC2030-IDC-NL" H 3200 3050 50  0001 C CNN
+F 3 "" H 3200 3050 50  0001 C CNN
+	1    3200 3050
+	-1   0    0    -1
+$EndComp
 Connection ~ 6250 2450
 Wire Wire Line
@@
 Connection ~ 7050 1850
 Connection ~ 4650 1850
+Wire Wire Line
+	3850 3250 3400 3250
+Wire Wire Line
+	3850 3150 3800 3150
+Wire Wire Line
+	3800 3150 3800 3050
+Wire Wire Line
+	3800 3050 3400 3050
+Wire Wire Line
+	3400 2950 3650 2950
+Wire Wire Line
+	3650 2950 3650 4050
+Wire Wire Line
+	3650 3150 3400 3150
+Connection ~ 3650 4050
+Connection ~ 3650 3150
+Wire Wire Line
+	3400 3350 3500 3350
+Wire Wire Line
+	3500 3350 3500 1850
+Connection ~ 3500 1850
+$Comp
+L GND #PWR02
+U 1 1 5AEE0D87
+P 4650 4050
+F 0 "#PWR02" H 4650 3800 50  0001 C CNN
+F 1 "GND" H 4650 3900 50  0000 C CNN
+F 2 "" H 4650 4050 50  0001 C CNN
+F 3 "" H 4650 4050 50  0001 C CNN
+	1    4650 4050
+	1    0    0    -1
+$EndComp
 $EndSCHEMATC

Commit message: Verified hole sizes WT51822, more pcb cleanup
Changed lines of the file:
@@
 Wire Wire Line
 	2650 4050 7050 4050
-Wire Wire Line
-	4650 3650 4650 4050
-Wire Wire Line
-	4450 3800 4850 3800
-Wire Wire Line
-	4850 3800 4850 3650
-Wire Wire Line
-	4750 3800 4750 3650
-Connection ~ 4750 3800
-Wire Wire Line
-	4450 3800 4450 3650
-Connection ~ 4650 3800
-Wire Wire Line
-	4550 3800 4550 3650
-Connection ~ 4550 3800
 $Comp
 L +3.3V #PWR01
@@
 	1    0    0    -1
 $EndComp
-Connection ~ 4650 4050
 $Comp
 L MMBT3904 Q1
@@
 Connection ~ 4650 1850
 Wire Wire Line
-	3850 3250 3400 3250
+	3700 3150 3850 3150
 Wire Wire Line
-	3850 3150 3800 3150
+	3400 2950 3600 2950
 Wire Wire Line
-	3800 3150 3800 3050
+	3600 2950 3600 4050
 Wire Wire Line
-	3800 3050 3400 3050
-Wire Wire Line
-	3400 2950 3650 2950
-Wire Wire Line
-	3650 2950 3650 4050
-Wire Wire Line
-	3650 3150 3400 3150
-Connection ~ 3650 4050
-Connection ~ 3650 3150
+	3600 3150 3400 3150
+Connection ~ 3600 4050
+Connection ~ 3600 3150
 Wire Wire Line
 	3400 3350 3500 3350
@@
 	1    0    0    -1
 $EndComp
+Wire Wire Line
+	3400 3250 3700 3250
+Wire Wire Line
+	3700 3250 3700 3150
+Wire Wire Line
+	3850 3250 3800 3250
+Wire Wire Line
+	3800 3250 3800 3050
+Wire Wire Line
+	3800 3050 3400 3050
+Wire Wire Line
+	4550 3650 4550 3800
+Wire Wire Line
+	4550 3800 4750 3800
+Wire Wire Line
+	4650 3650 4650 4050
+Wire Wire Line
+	4750 3800 4750 3650
+Connection ~ 4650 3800
+Connection ~ 4650 4050
 $EndSCHEMATC

Commit message: As sent to pcbway 20180517
Parts:
- BT1: symbol Battery_Cell -> device:Battery_Cell
- J1: symbol Conn_01x06 -> conn:Conn_01x06
- Q1: symbol MMBT3904 -> transistors:MMBT3904
- R1, R2, R3: symbol R -> device:R
- S1: symbol FibretronicKeypad -> fibretronickeypad:FibretronicKeypad
- U1: symbol WT51822-0S4AT -> WT51822-0S4AT:WT51822-0S4AT
Changed lines of the file:
@@
-EESchema Schematic File Version 2
-LIBS:power
-LIBS:device
-LIBS:switches
-LIBS:relays
-LIBS:motors
-LIBS:transistors
-LIBS:conn
-LIBS:linear
-LIBS:regul
-LIBS:74xx
-LIBS:cmos4000
-LIBS:adc-dac
-LIBS:memory
-LIBS:xilinx
-LIBS:microcontrollers
-LIBS:dsp
-LIBS:microchip
-LIBS:analog_switches
-LIBS:motorola
-LIBS:texas
-LIBS:intel
-LIBS:audio
-LIBS:interface
-LIBS:digital-audio
-LIBS:philips
-LIBS:display
-LIBS:cypress
-LIBS:siliconi
-LIBS:opto
-LIBS:atmel
-LIBS:contrib
-LIBS:valves
-LIBS:WT51822-0S4AT
-LIBS:fibretronickeypad
+EESchema Schematic File Version 4
 LIBS:wearlink-cache
-EELAYER 25 0
+EELAYER 26 0
 EELAYER END
 $Descr A4 11693 8268
@@
 $EndDescr
 $Comp
-L WT51822-0S4AT U1
+L WT51822-0S4AT:WT51822-0S4AT U1
 U 1 1 5AED8A82
 P 4650 2850
@@
 $EndComp
 $Comp
-L Battery_Cell BT1
+L device:Battery_Cell BT1
 U 1 1 5AED9A99
 P 2650 2950
@@
 	2650 2750 2650 1850
 Wire Wire Line
-	2650 1850 7750 1850
+	2650 1850 3500 1850
 Wire Wire Line
 	4650 1850 4650 2050
@@
 	2650 3050 2650 4050
 Wire Wire Line
-	2650 4050 7050 4050
-$Comp
-L +3.3V #PWR01
+	2650 4050 3600 4050
+$Comp
+L power:+3.3V #PWR01
 U 1 1 5AEDB4DB
 P 4650 1850
@@
 $EndComp
 $Comp
-L FibretronicKeypad S1
+L fibretronickeypad:FibretronicKeypad S1
 U 1 1 5AEDB75E
 P 8650 2350
@@
 $EndComp
 $Comp
-L R R1
+L device:R R1
 U 1 1 5AEDBA85
 P 6250 3550
-F 0 "R1" V 6330 3550 50  0000 C CNN
+F 0 "R1" H 6350 3550 50  0000 C CNN
 F 1 "20k" V 6250 3550 50  0000 C CNN
 F 2 "Resistors_SMD:R_0603" V 6180 3550 50  0001 C CNN
@@
 $EndComp
 $Comp
-L MMBT3904 Q1
+L transistors:MMBT3904 Q1
 U 1 1 5AEDBB1B
 P 6950 3200
@@
 $EndComp
 $Comp
-L R R3
+L device:R R3
 U 1 1 5AEDBDFB
 P 7050 2150
-F 0 "R3" V 7130 2150 50  0000 C CNN
+F 0 "R3" H 7150 2150 50  0000 C CNN
 F 1 "1M" V 7050 2150 50  0000 C CNN
 F 2 "Resistors_SMD:R_0603" V 6980 2150 50  0001 C CNN
@@
 $EndComp
 $Comp
-L R R2
+L device:R R2
 U 1 1 5AEDBE6E
 P 6500 3200
@@
 	6650 3200 6750 3200
 Wire Wire Line
-	7050 2300 7050 3000
+	7050 2300 7050 2750
 Wire Wire Line
 	7050 1850 7050 2000
 Wire Wire Line
-	6250 2450 6250 3400
+	6250 2450 6250 3200
 Connection ~ 7050 2750
 Connection ~ 6250 3200
@@
 	5450 2750 7050 2750
 Wire Wire Line
-	5450 2450 7750 2450
+	5450 2450 6250 2450
 Wire Wire Line
 	6350 3200 6250 3200
@@
 POWER
 $Comp
-L Conn_01x06 J1
+L conn:Conn_01x06 J1
 U 1 1 5AEDCC20
 P 3200 3050
@@
 	3400 2950 3600 2950
 Wire Wire Line
-	3600 2950 3600 4050
+	3600 2950 3600 3150
 Wire Wire Line
 	3600 3150 3400 3150
@@
 Connection ~ 3500 1850
 $Comp
-L GND #PWR02
+L power:GND #PWR02
 U 1 1 5AEE0D87
 P 4650 4050
@@
 	4550 3650 4550 3800
 Wire Wire Line
-	4550 3800 4750 3800
-Wire Wire Line
-	4650 3650 4650 4050
+	4550 3800 4650 3800
+Wire Wire Line
+	4650 3650 4650 3800
 Wire Wire Line
 	4750 3800 4750 3650
 Connection ~ 4650 3800
 Connection ~ 4650 4050
+Wire Wire Line
+	6250 4050 7050 4050
+Wire Wire Line
+	7050 2750 7050 3000
+Wire Wire Line
+	6250 3200 6250 3400
+Wire Wire Line
+	6250 2450 7750 2450
+Wire Wire Line
+	7050 1850 7750 1850
+Wire Wire Line
+	4650 1850 7050 1850
+Wire Wire Line
+	3600 4050 4650 4050
+Wire Wire Line
+	3600 3150 3600 4050
+Wire Wire Line
+	3500 1850 4650 1850
+Wire Wire Line
+	4650 3800 4750 3800
+Wire Wire Line
+	4650 3800 4650 4050
+Wire Wire Line
+	4650 4050 6250 4050
 $EndSCHEMATC
